File: PCB_Rev2/Multi/PH60_Rev2.kicad_pcb (KiCad board)
At the start: 2 copper layers, 285 x 94.6 mm, 182 parts, among them J1 USB_C_Receptacle_USB2.0_16P, J2 Conn_01x02, U2 W25Q128JVS, U3 RP2040, U4 XC6206PxxxMR, Y1 Crystal_GND24

Commit message: Multi PCB Update
Parts:
- removed the S14 at (285.8, 38.1)
- removed the S28 at (281.0, 76.2)
- removed the S28 at (300.0, 57.1)
- removed the S29 at (40.5, 76.2)
- removed the S29 at (45.2, 76.2)
- removed the S41 at (302.4, 66.7)
- removed the S41 at (292.9, 76.2)
- removed the S43 at (50.0, 95.2)
- removed the S55 at (288.1, 95.2)
- removed the S55 at (278.6, 95.2)
- removed the S57 at (42.9, 114.3)
- removed the S57 at (40.5, 114.3)
- removed the S58 at (66.7, 114.3)
- removed the S58 at (64.3, 114.3)
- removed the S59 at (88.1, 114.3)
- removed the S59 at (90.5, 114.3)
- removed the S60 at (171.4, 114.3)
- removed the S62 at (252.4, 114.3)
- removed the S62 at (254.8, 114.3)
- removed the S63 at (276.2, 114.3)
- removed the S63 at (278.6, 114.3)
- removed the S64 at (302.4, 114.3)
- removed the S64 at (300.0, 114.3)
- added D65: PRTR5V0U2X, Package_TO_SOT_SMD:SOT-143, B.Cu at (49.2, 39.8)
- added S14-2: MX1A, PCM_Switch_Keyboard_Hotswap_Kailh:SW_Hotswap_Kailh_MX_Plated_1.00u, F.Cu at (304.8, 38.1)
- added S28: MX1A, PCM_Switch_Keyboard_Hotswap_Kailh:SW_Hotswap_Kailh_MX_Plated_ISOEnter_90deg, F.Cu at (302.4, 66.7)
- added S28-2: MX1A, PCM_Switch_Keyboard_Hotswap_Kailh:SW_Hotswap_Kailh_MX_Plated_1.50u_90deg, F.Cu at (300.0, 57.1)
- added S29: MX1A, PCM_Switch_Keyboard_Hotswap_Kailh:SW_Hotswap_Kailh_MX_Plated_1.75u, F.Cu at (45.2, 76.2)
- added S29-2: MX1A, PCM_Switch_Keyboard_Hotswap_Kailh:SW_Hotswap_Kailh_MX_Plated_1.25u, F.Cu at (40.5, 76.2)
- added S41: MX1A, PCM_Switch_Keyboard_Hotswap_Kailh:SW_Hotswap_Kailh_MX_Plated_1.00u, F.Cu at (281.0, 76.2)
- added S41-2: MX1A, PCM_Switch_Keyboard_Hotswap_Kailh:SW_Hotswap_Kailh_MX_Plated_2.25u_90deg, F.Cu at (292.9, 76.2)
- added S43-2: MX1A, PCM_Switch_Keyboard_Hotswap_Kailh:SW_Hotswap_Kailh_MX_Plated_2.25u, F.Cu at (50.0, 95.2)
- added S55: MX1A, PCM_Switch_Keyboard_Hotswap_Kailh:SW_Hotswap_Kailh_MX_Plated_1.75u, F.Cu at (278.6, 95.2)
- added S55-2: MX1A, PCM_Switch_Keyboard_Hotswap_Kailh:SW_Hotswap_Kailh_MX_Plated_2.75u, F.Cu at (288.1, 95.2)
- added S57: MX1A, PCM_Switch_Keyboard_Hotswap_Kailh:SW_Hotswap_Kailh_MX_Plated_1.25u, F.Cu at (40.5, 114.3)
- added S57-2: MX1A, PCM_Switch_Keyboard_Hotswap_Kailh:SW_Hotswap_Kailh_MX_Plated_1.50u, F.Cu at (42.9, 114.3)
- added S58: MX1A, PCM_Switch_Keyboard_Hotswap_Kailh:SW_Hotswap_Kailh_MX_Plated_1.25u, F.Cu at (64.3, 114.3)
- added S58-2: MX1A, PCM_Switch_Keyboard_Hotswap_Kailh:SW_Hotswap_Kailh_MX_Plated_1.00u, F.Cu at (66.7, 114.3)
- added S59: MX1A, PCM_Switch_Keyboard_Hotswap_Kailh:SW_Hotswap_Kailh_MX_Plated_1.25u, F.Cu at (88.1, 114.3)
- added S59-2: MX1A, PCM_Switch_Keyboard_Hotswap_Kailh:SW_Hotswap_Kailh_MX_Plated_1.50u, F.Cu at (90.5, 114.3)
- added S60-2: MX1A, PCM_Switch_Keyboard_Hotswap_Kailh:SW_Hotswap_Kailh_MX_Plated_7.00u, F.Cu at (171.4, 114.3)
- added S61-2: MX1A, PCM_Switch_Keyboard_Hotswap_Kailh:SW_Hotswap_Kailh_MX_Plated_1.50u, F.Cu at (252.4, 114.3)
- added S62: MX1A, PCM_Switch_Keyboard_Hotswap_Kailh:SW_Hotswap_Kailh_MX_Plated_1.25u, F.Cu at (254.8, 114.3)
- added S62-2: MX1A, PCM_Switch_Keyboard_Hotswap_Kailh:SW_Hotswap_Kailh_MX_Plated_1.00u, F.Cu at (276.2, 114.3)
- added S63: MX1A, PCM_Switch_Keyboard_Hotswap_Kailh:SW_Hotswap_Kailh_MX_Plated_1.25u, F.Cu at (278.6, 114.3)
- added S64: MX1A, PCM_Switch_Keyboard_Hotswap_Kailh:SW_Hotswap_Kailh_MX_Plated_1.25u, F.Cu at (302.4, 114.3)
- added S64-2: MX1A, PCM_Switch_Keyboard_Hotswap_Kailh:SW_Hotswap_Kailh_MX_Plated_1.50u, F.Cu at (300.0, 114.3)
- C1, C4: value 10u -> 1u
- J2: footprint Connector_PinHeader_2.54mm:PinHeader_1x02_P2.54mm_Vertical -> Connector_PinHeader_1.27mm:PinHeader_1x02_P1.27mm_Vertical
- U2: footprint Package_SO:SOIC-8_5.23x5.23mm_P1.27mm -> Package_SON:Winbond_USON-8-1EP_3x2mm_P0.5mm_EP0.2x1.6mm
- U3: footprint Package_DFN_QFN:QFN-56-1EP_7x7mm_P0.4mm_EP3.2x3.2mm_ThermalVias -> Package_DFN_QFN:QFN-56-1EP_7x7mm_P0.4mm_EP3.2x3.2mm
- moved D58 22.8 mm to (76.7, 107.6)
- moved D59 22.8 mm to (100.5, 107.6)
- moved S42 19.1 mm to (285.8, 38.1)
- moved C14 18.9 mm to (137.3, 107.2), turned to 90 degrees
- moved D43 17.3 mm to (67.0, 98.5), turned to 90 degrees
- moved D42 15.9 mm to (284.0, 57.1), turned to 90 degrees
- moved C9 14.6 mm to (130.9, 118.1), turned to -90 degrees
- moved C5 14.3 mm to (124.9, 109.3), turned to 180 degrees
- moved D55 11.4 mm to (266.6, 100.1)
- moved U4 10.8 mm to (119.0, 109.3)
- moved C1 10.6 mm to (115.9, 109.8)
- moved D56 10.6 mm to (309.9, 92.0), turned to -90 degrees
- moved C16 10.5 mm to (129.4, 113.6)
- moved J2 10.4 mm to (125.7, 107.0)
- moved C12 9.55 mm to (136.4, 118.6), turned to 180 degrees
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Connections:
- S42 pad 1: Net-(D42-A) -> col_13
- S42 pad 2: col_13 -> Net-(D42-A)
- U3 pad 27: row_2 -> unconnected-(U3-GPIO16-Pad27)
- U3 pad 28: row_3 -> unconnected-(U3-GPIO17-Pad28)
- U3 pad 29: row_4 -> row_2
- U3 pad 30: unconnected-(U3-GPIO19-Pad30) -> row_3
- U3 pad 31: unconnected-(U3-GPIO20-Pad31) -> row_4
Routing:
- net row_0: track 396.2 -> 322.2 mm
- net row_1: track 371.0 -> 300.9 mm
- net row_2: track 330.3 -> 290.8 mm, vias 4 -> 2
- net row_3: track 307.8 -> 276.0 mm, vias 2 -> 0
- net GND: track 43.5 -> 72.9 mm, vias 52 -> 19
- net Net-(D28-A): track 77.3 -> 49.5 mm
- net Net-(D62-A): track 16.2 -> 41.5 mm
- net col_12: track 275.3 -> 299.2 mm
- net col_10: track 186.5 -> 209.4 mm
- net Net-(D61-A): track 5.09 -> 26.8 mm
- net col_11: track 234.3 -> 254.5 mm
- net Net-(D14-A): track 15.5 -> 35.1 mm
- net +3V3: track 86.0 -> 66.7 mm, vias 5 -> 4
- net /~{USB_BOOT}: track 18.1 -> 1.74 mm, vias 1 -> 0
- net VBUS: track 152.8 -> 169.1 mm, vias 2 -> 3
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Other:
- board text added: "By Team PHDesign M_Altmann nonameC_ alt-0191"
- board text added: "PH60/Multi"
