File: PCB_Rev2/Multi/PH60_Rev2.kicad_sch (KiCad schematic)
At the start: 28 parts, among them J1 USB_C_Receptacle_USB2.0_16P, J2 Conn_01x02, U2 W25Q128JVS, U3 RP2040, U4 XC6206PxxxMR, Y1 Crystal_GND24

Commit message: Multi PCB Update
Parts:
- added D65: PRTR5V0U2X, Package_TO_SOT_SMD:SOT-143, symbol Power_Protection:PRTR5V0U2X
- added U1: ~, nRF_Module:nRF52810_Module, symbol nRF52810_Module:LC52810
- C1, C4: value 10u -> 1u
- J2: footprint Connector_PinHeader_2.54mm:PinHeader_1x02_P2.54mm_Vertical -> Connector_PinHeader_1.27mm:PinHeader_1x02_P1.27mm_Vertical
- U2: footprint Package_SO:SOIC-8_5.23x5.23mm_P1.27mm -> Package_SON:Winbond_USON-8-1EP_3x2mm_P0.5mm_EP0.2x1.6mm
- U3: footprint Package_DFN_QFN:QFN-56-1EP_7x7mm_P0.4mm_EP3.2x3.2mm_ThermalVias -> Package_DFN_QFN:QFN-56-1EP_7x7mm_P0.4mm_EP3.2x3.2mm
Connections:
- net GND: now also D65.1 (GND)
- net USB_D+: now also D65.2 (I/O1)
- net USB_D-: now also D65.3 (I/O2)
- net VBUS: now also D65.4 (VCC)
- net row_2: now also U3.29 (GPIO18); no longer U3.27 (GPIO16)
- net row_3: now also U3.30 (GPIO19); no longer U3.28 (GPIO17)
- net row_4: now also U3.31 (GPIO20); no longer U3.29 (GPIO18)
