File: PCB_Rev2/Multi/matrix.kicad_sch (KiCad schematic)
At the start: 128 parts

Commit message: Multi PCB Update
Parts:
- added S14-2, S58-2, S62-2: MX1A, PCM_Switch_Keyboard_Hotswap_Kailh:SW_Hotswap_Kailh_MX_Plated_1.00u, symbol Switch:SW_Push
- added S28-2: MX1A, PCM_Switch_Keyboard_Hotswap_Kailh:SW_Hotswap_Kailh_MX_Plated_1.50u_90deg, symbol Switch:SW_Push
- added S29-2: MX1A, PCM_Switch_Keyboard_Hotswap_Kailh:SW_Hotswap_Kailh_MX_Plated_1.25u, symbol Switch:SW_Push
- added S41-2: MX1A, PCM_Switch_Keyboard_Hotswap_Kailh:SW_Hotswap_Kailh_MX_Plated_2.25u_90deg, symbol Switch:SW_Push
- added S43-2: MX1A, PCM_Switch_Keyboard_Hotswap_Kailh:SW_Hotswap_Kailh_MX_Plated_2.25u, symbol Switch:SW_Push
- added S55-2: MX1A, PCM_Switch_Keyboard_Hotswap_Kailh:SW_Hotswap_Kailh_MX_Plated_2.75u, symbol Switch:SW_Push
- added S57-2, S59-2, S61-2, S64-2: MX1A, PCM_Switch_Keyboard_Hotswap_Kailh:SW_Hotswap_Kailh_MX_Plated_1.50u, symbol Switch:SW_Push
- added S60-2: MX1A, PCM_Switch_Keyboard_Hotswap_Kailh:SW_Hotswap_Kailh_MX_Plated_7.00u, symbol Switch:SW_Push
- S28: footprint PCM_Switch_Keyboard_Hotswap_Kailh:SW_Hotswap_Kailh_MX_Plated_1.50u_90deg -> PCM_Switch_Keyboard_Hotswap_Kailh:SW_Hotswap_Kailh_MX_Plated_ISOEnter_90deg
- S29: footprint PCM_Switch_Keyboard_Hotswap_Kailh:SW_Hotswap_Kailh_MX_Plated_1.75u_90deg -> PCM_Switch_Keyboard_Hotswap_Kailh:SW_Hotswap_Kailh_MX_Plated_1.75u
- S41: footprint PCM_Switch_Keyboard_Hotswap_Kailh:SW_Hotswap_Kailh_MX_Plated_2.25u_90deg -> PCM_Switch_Keyboard_Hotswap_Kailh:SW_Hotswap_Kailh_MX_Plated_1.00u
- S43: renamed from S42; footprint PCM_Switch_Keyboard_Hotswap_Kailh:SW_Hotswap_Kailh_MX_Plated_2.25u -> PCM_Switch_Keyboard_Hotswap_Kailh:SW_Hotswap_Kailh_MX_Plated_1.25u
- S55: footprint PCM_Switch_Keyboard_Hotswap_Kailh:SW_Hotswap_Kailh_MX_Plated_2.75u_90deg -> PCM_Switch_Keyboard_Hotswap_Kailh:SW_Hotswap_Kailh_MX_Plated_1.75u
- S57: renamed from S55; footprint PCM_Switch_Keyboard_Hotswap_Kailh:SW_Hotswap_Kailh_MX_Plated_1.25u_90deg -> PCM_Switch_Keyboard_Hotswap_Kailh:SW_Hotswap_Kailh_MX_Plated_1.25u
- S58: renamed from S56; footprint PCM_Switch_Keyboard_Hotswap_Kailh:SW_Hotswap_Kailh_MX_Plated_1.25u_90deg -> PCM_Switch_Keyboard_Hotswap_Kailh:SW_Hotswap_Kailh_MX_Plated_1.25u
- S59: renamed from S57; footprint PCM_Switch_Keyboard_Hotswap_Kailh:SW_Hotswap_Kailh_MX_Plated_1.25u_90deg -> PCM_Switch_Keyboard_Hotswap_Kailh:SW_Hotswap_Kailh_MX_Plated_1.25u
- S62: renamed from S60; footprint PCM_Switch_Keyboard_Hotswap_Kailh:SW_Hotswap_Kailh_MX_Plated_1.25u_90deg -> PCM_Switch_Keyboard_Hotswap_Kailh:SW_Hotswap_Kailh_MX_Plated_1.25u
- S63: renamed from S61; footprint PCM_Switch_Keyboard_Hotswap_Kailh:SW_Hotswap_Kailh_MX_Plated_1.25u_90deg -> PCM_Switch_Keyboard_Hotswap_Kailh:SW_Hotswap_Kailh_MX_Plated_1.25u
- S64: renamed from S62; footprint PCM_Switch_Keyboard_Hotswap_Kailh:SW_Hotswap_Kailh_MX_Plated_1.25u_90deg -> PCM_Switch_Keyboard_Hotswap_Kailh:SW_Hotswap_Kailh_MX_Plated_1.25u
- renumbered D42 to D43, D43 to D44, D46 to D47, D47 to D48, D48 to D49, D49 to D50, D50 to D51, D51 to D52, D52 to D53, D55 to D57, D56 to D58, D57 to D59, D58 to D60, D59 to D61, D60 to D62, D61 to D63, D62 to D64, S43 to S44, S46 to S47, S47 to S48, S48 to S49, S49 to S50, S50 to S51, S51 to S52, S52 to S53, S58 to S60, S59 to S61
Connections:
- net col_0: now also S43.1, S57.1, S29-2.1, S43-2.2, S57-2.2; no longer S43.2, S57.2
- net col_1: now also S58.1, S58-2.2; no longer S58.2
- net col_10: now also S61-2.2
- net col_11: now also S62.1, S62-2.2; no longer S62.2
- net col_12: now also S28.2, S55.1, S63.1, S41-2.2, S55-2.2; no longer S41.2, S55.2, S63.2
- net col_13: now also S41.2, S42.1, S64.1, S14-2.2, S28-2.1, S64-2.2; no longer S28.2, S42.2, S64.2
- net col_2: now also S59.1, S59-2.2; no longer S59.2
- net col_6: now also S60-2.1
- net at D64.2 (A): now also S64.2, S64-2.1; no longer S64.1
- net at D14.2 (A), S14.1: now also S14-2.1
- net at D58.2 (A): now also S58.2, S58-2.1; no longer S58.1
- net at D43.2 (A): now also S43.2, S43-2.1; no longer S43.1
- net at D62.2 (A): now also S62.2, S62-2.1; no longer S62.1
- net at D60.2 (A), S60.1: now also S60-2.2
- net at S28.1: now also D41.2 (A), S41-2.1; no longer D28.2 (A)
- net at D59.2 (A): now also S59.2, S59-2.1; no longer S59.1
- net at D55.2 (A): now also S55.2, S55-2.1; no longer S55.1
- net at D63.2 (A): now also S63.2; no longer S63.1
- net at D42.2 (A): now also S42.2; no longer S42.1
- net at D61.2 (A), S61.1: now also S61-2.1
- net at D57.2 (A): now also S57.2, S57-2.1; no longer S57.1
- net at S41.1: now also D28.2 (A), S28-2.2; no longer D41.2 (A)
- net at D29.2 (A), S29.1: now also S29-2.2
Other:
- moved on the sheet: S28, S41, S42, S43, S55, S57, S58, S59, S62, S63, S64
